File: pcb/imperializer.sch (KiCad schematic (older format))
At the start: 24 parts, among them J1 USB_micro_horz_socket_reinfor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, J2 Conn_01x06_Male, SW1 SW_SPST, U1 AS1115-BSST, U2 ATMEGA32U4, U3 LTC-4727, U4 LTC-4727, U5 AP7313, X1 AVR_ISP, Y1 Resonator

Commit message: pcb v1.1
Parts:
- removed J1: USB_micro_horz_socket_reinforced, asl_footprints:microUSB_horizontal_socket, symbol asl_symbols:USB_micro_horz_socket_reinforced
- removed J2: Conn_01x06_Male, Connector_PinHeader_2.54mm:PinHeader_1x06_P2.54mm_Vertical, symbol Connector:Conn_01x06_Male
- removed U2: ATMEGA32U4, Package_QFP:TQFP-44_10x10mm_P0.8mm, symbol asl_symbols:ATMEGA32U4
- removed U5: AP7313, Package_TO_SOT_SMD:TSOT-23, symbol asl_symbols:AP7313
- removed X1: AVR_ISP, asl_footprints:AVR_ISP, symbol asl_symbols:AVR_ISP
- removed Y1: Resonator, Crystal:Resonator_SMD_muRata_CSTxExxV-3Pin_3.0x1.1mm, symbol asl_symbols:Resonator
- added BT1, BT2: Battery, Battery:BatteryHolder_Keystone_2466_1xAAA, symbol Device:Battery
- added H1, H2, H3, H4: Threaded_Standoff, asl_footprints:standoff_nut, symbol asl_symbols:Threaded_Standoff
- added R4, R5, R6, R7, R8, R9: 10KΩ, Resistor_SMD:R_0805_2012Metric, symbol Device:R_Small_US
- added U4: trinket_M0, asl_footprints:trinket_M0, symbol asl_symbols:trinket_M0
- added U6, U7: LTC-4727, asl_footprints:LTC-4727, symbol asl_symbols:LTC-4727
- added U8: AS1115-BSST, Package_SO:QSOP-24_3.9x8.7mm_P0.635mm, symbol asl_symbols:AS1115-BSST
- R1, R2: value 27Ω -> 10KΩ
- R3: value 25KΩ -> 10KΩ
- S1: renamed from S9; symbol asl_symbols:switch_momentary_2pin -> imperializer-rescue:switch_momentary_2pin-asl_symbols; Description (none) -> Gateron Blue Key Switch
- S10: renamed from S7; symbol asl_symbols:switch_momentary_2pin -> imperializer-rescue:switch_momentary_2pin-asl_symbols; Description (none) -> Gateron Blue Key Switch
- S11: renamed from S8; symbol asl_symbols:switch_momentary_2pin -> imperializer-rescue:switch_momentary_2pin-asl_symbols; Description (none) -> Gateron Blue Key Switch
- S2: renamed from S10; symbol asl_symbols:switch_momentary_2pin -> imperializer-rescue:switch_momentary_2pin-asl_symbols; Description (none) -> Gateron Blue Key Switch
- S3: renamed from S11; symbol asl_symbols:switch_momentary_2pin -> imperializer-rescue:switch_momentary_2pin-asl_symbols; Description (none) -> Gateron Blue Key Switch
- S4: renamed from S1; symbol asl_symbols:switch_momentary_2pin -> imperializer-rescue:switch_momentary_2pin-asl_symbols; Description (none) -> Gateron Blue Key Switch
- S5: renamed from S2; symbol asl_symbols:switch_momentary_2pin -> imperializer-rescue:switch_momentary_2pin-asl_symbols; Description (none) -> Gateron Blue Key Switch
- S6: renamed from S3; symbol asl_symbols:switch_momentary_2pin -> imperializer-rescue:switch_momentary_2pin-asl_symbols; Description (none) -> Gateron Blue Key Switch
- S7: renamed from S4; symbol asl_symbols:switch_momentary_2pin -> imperializer-rescue:switch_momentary_2pin-asl_symbols; Description (none) -> Gateron Blue Key Switch
- S8: renamed from S5; symbol asl_symbols:switch_momentary_2pin -> imperializer-rescue:switch_momentary_2pin-asl_symbols; Description (none) -> Gateron Blue Key Switch
- S9: renamed from S6; symbol asl_symbols:switch_momentary_2pin -> imperializer-rescue:switch_momentary_2pin-asl_symbols; Description (none) -> Gateron Blue Key Switch
- renumbered U4 to U2, U1 to U5
Connections:
- net GND: now also BT2.2 (-), U4.2 (GND), U8.6 (GND)
- net IRQ: now also R1.2, U4.3 (4)
- net SCL: now also R6.1, U4.7 (2), U8.14 (SCL)
- net SDA: now also R5.1, U4.9 (0), U8.1 (SDA)
- net mode: now also U4.4 (3)
- net at U5.13 (ISET): now also R4.1; no longer R3.2
- net at R2.1: now also R3.1, R4.2
- net VBATT: now reaches R1.1
- net VBATT: now also R2.2, R3.2, U5.19 (VDD), BT1.1 (+), R5.2, R6.2, R7.2, R8.2, U4.1 (BAT), U8.19 (VDD)
- removed net 3.3VDC: R3.1, U5.19 (VDD)
- new net: R9.1, U8.13 (ISET)
- new net: BT1.2 (-), BT2.1 (+)
- new net: R7.1, R8.1, R9.2
- new net DIG0-2: U6.1 (D1), U8.2 (DIG0)
- new net DIG1-2: U6.2 (D2), U8.3 (DIG1)
- new net DIG2-2: U6.6 (D3), U8.4 (DIG2)
- new net DIG3-2: U6.8 (D4), U8.5 (DIG3)
- new net DIG4-2: U7.1 (D1), U8.7 (DIG4)
- new net DIG5-2: U7.2 (D2), U8.8 (DIG5)
- new net DIG6-2: U7.6 (D3), U8.9 (DIG6)
- new net DIG7-2: U7.8 (D4), U8.10 (DIG7)
- new net a2: U6.14 (a), U7.14 (a), U8.15 (SEGA)
- new net b2: U6.16 (b), U7.16 (b), U8.17 (SEGB)
- new net c2: U6.13 (c), U7.13 (c), U8.20 (SEGC)
- new net d2: U6.3 (d), U7.3 (d), U8.23 (SEGD)
- new net dp2: U6.7 (DPX), U7.7 (DPX), U8.22 (SEGDP)
- new net e2: U6.5 (e), U7.5 (e), U8.21 (SEGE)
- new net f2: U6.11 (f), U7.11 (f), U8.11 (KEYA), U8.16 (SEGF)
- new net g2: U6.15 (g), U7.15 (g), U8.18 (SEGG)
- no-connect marks 2 -> 4
Other:
- moved on the sheet: S1, S10, S11, S2, S3, S4, S5, S6, S7, S8, S9, SW1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

Commit message: pcb v1.2
switched to bare SAMD21
added USB-C connector
added 4 conversion selection LEDs
added on/off button with soft latch circuit
rearranged toggles switch and battery holders
Parts:
- removed U4: trinket_M0, asl_footprints:trinket_M0, symbol asl_symbols:trinket_M0
- added C1, C2: 15pF, Capacitor_SMD:C_0805_2012Metric, symbol Device:C
- added C3, C4: 0.1µF, Capacitor_SMD:C_0805_2012Metric, symbol Device:C
- added C5: 10nF, Capacitor_SMD:C_0805_2012Metric, symbol Device:C
- added D1, D3: BAT54C, Package_TO_SOT_SMD:SOT-23, symbol Diode:BAT54C
- added D2, D4, D5, D6, D7, D8: LED, LED_SMD:LED_0805_2012Metric, symbol Device:LED
- added J1: USB_C_Receptacle_USB2.0, asl_footprints:USB_C_Receptacle_GCT_USB4085, symbol asl_symbols:USB_C_Receptacle_USB2.0
- added J2: SWD_connector, asl_footprints:SWD_2x5_socket, symbol asl_symbols:SWD_connector
- added Q1, Q3: FDN340P, Package_TO_SOT_SMD:SOT-23, symbol asl_symbols:FDN340P
- added Q2: BSS123, Package_TO_SOT_SMD:SOT-23, symbol Transistor_FET:BSS123
- added R10, R18, R19, R20, R21: 10KΩ, Resistor_SMD:R_0805_2012Metric, symbol Device:R_Small_US
- added R11: 100KΩ, Resistor_SMD:R_0805_2012Metric, symbol Device:R_Small_US
- added R12, R16, R17: 330KΩ, Resistor_SMD:R_0805_2012Metric, symbol Device:R_Small_US
- added R13: 1MΩ, Resistor_SMD:R_0805_2012Metric, symbol Device:R_Small_US
- added R14, R15: 5.1KΩ, Resistor_SMD:R_0805_2012Metric, symbol Device:R_Small_US
- added S12, S13: B3FS-1010P, asl_footprints:6mm_tactile_smd, symbol asl_symbols:B3FS-1010P
- added U1: ATSAMD21G15A-A, Package_QFP:TQFP-48_7x7mm_P0.5mm, symbol MCU_Microchip_SAMD:ATSAMD21G15A-A
- added U4: AP2112K-3.3, Package_TO_SOT_SMD:SOT-23-5, symbol asl_symbols:AP2112K-3.3
- added U9: LTC4412xS6, Package_TO_SOT_SMD:TSOT-23-6, symbol Power_Management:LTC4412xS6
- added Y1: Crystal, Crystal:Crystal_SMD_0603-2Pin_6.0x3.5mm, symbol Device:Crystal
- S1, S10, S11, S2, S3, S4, S5, S6, S7, S8, S9: symbol imperializer-rescue:switch_momentary_2pin-asl_symbols -> imperializer-rescue:switch_momentary_2pin-asl_symbols-imperializer-rescue
- SW1: footprint Connector_PinHeader_2.54mm:PinHeader_1x03_P2.54mm_Vertical -> asl_footprints:B12AP
Connections:
- net GND: now also C1.2, C2.1, C3.1, C4.2, D4.1 (K), D5.1 (K), D6.1 (K), D7.1 (K), D8.1 (K), J1.A1 (GND), J1.A12 (GND), J1.B1 (GND), J1.B12 (GND), J1.S1 (SHIELD), J2.3 (GND), J2.5 (GND), J2.9 (GNDDetect), Q2.2 (S), R13.1, R14.2, R15.2, S12.4 (out2), S13.3 (out1), S13.4 (out2), U1.18 (GND), U1.35 (GND), U1.42 (GND), U1.5 (GNDANA), U4.2 (GND), U9.2 (GND), U9.3 (CTL)
- net IRQ: now also U1.11 (PA06)
- net SCL: now also U1.32 (PA23)
- net SDA: now also U1.31 (PA22)
- net VBATT: now also C5.1, Q1.2 (S), R11.2; no longer R1.1, R2.2, R3.2, R5.2, R6.2, R7.2, R8.2, U5.19 (VDD), U8.19 (VDD)
- net mode: now also U1.12 (PA07)
- new net: D1.3, S12.2 (in2)
- new net: C1.1, U1.1 (PA00), Y1.2
- new net: C2.2, U1.2 (PA01), Y1.1
- new net: R18.1, U1.25 (PA16)
- new net: R19.1, U1.26 (PA17)
- new net: R20.1, U1.27 (PA18)
- new net: R21.1, U1.28 (PA19)
- new net: C3.2, U1.43 (VDDCORE)
- new net: D1.1, Q2.1 (G), R12.2, R13.2
- new net: C5.2, D1.2, Q1.1 (G), Q2.3 (D), R11.1
- new net: Q1.3 (D), Q3.2 (S), U9.1 (VIN)
- new net: D3.3, U4.1 (VIN), U4.3 (EN)
- new net: J1.A5 (CC1), R14.1
- new net: J1.B5 (CC2), R15.1
- new net: D2.1 (K), U9.4 (STAT)
- new net: Q3.1 (G), U9.5 (GATE)
- new net: D2.2 (A), R16.2
- new net: D4.2 (A), R17.2
- new net: D8.2 (A), R21.2
- new net: D7.2 (A), R20.2
- new net: D6.2 (A), R19.2
- new net: D5.2 (A), R18.2
- new net BTN: R12.1, U1.3 (PA02)
- new net D+: J1.A6 (D+), J1.B6 (D+), U1.34 (PA25)
- new net D-: J1.A7 (D-), J1.B7 (D-), U1.33 (PA24)
- new net RST: J2.10 (~RESET~), R10.1, S13.1 (in1), S13.2 (in2), U1.40 (~RESET)
- new net SWCLK: J2.4 (SWDCLK/TCK), U1.45 (PA30)
- new net SWDIO: J2.2 (SWDIO/TMS), U1.46 (PA31)
- new net VIN: C4.1, J2.1 (VTref), Q3.3 (D), R1.1, R10.2, R16.1, R17.1, R2.2, R3.2, R5.2, R6.2, R7.2, R8.2, U1.17 (VDDIO), U1.36 (VDDIO), U1.44 (VDDIN), U1.6 (VDDANA), U4.5 (VOUT), U5.19 (VDD), U8.19 (VDD), U9.6 (SENSE)
- new net VUSB: D3.1, J1.A4 (VBUS), J1.A9 (VBUS), J1.B4 (VBUS), J1.B9 (VBUS)
Other:
- note added: "Soft latch circuit with button input\nhttps://hackaday.com/2019/06/24/ditch-the-switch-a-soft-latching-circuit-roundup/\nhttps://youtu.be/7D9L9oS4AJM?t=683"
- moved on the sheet: BT1, BT2, H1, H2, H3, H4, R1, R2, R3, R4, R5, R6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
