File: pcb/imperializer.kicad_sch (KiCad schematic)
At the start: 69 parts, among them J1 USB_C_Receptacle_USB2.0, J2 SWD_connector, Q1 FDN340P, Q2 BSS123, Q3 FDN340P, SW1 SW_SPST, U1 ATSAMD21G15A-A, U2 LTC-4727, U3 LTC-4727, U4 AP2112K-3.3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

Commit message: pcb v1.3
Parts:
- removed BT2: Battery, Battery:BatteryHolder_Keystone_2466_1xAAA, symbol Device:Battery
- removed C1, C2: 15pF, Capacitor_SMD:C_0805_2012Metric, symbol Device:C
- removed D3: BAT54C, Package_TO_SOT_SMD:SOT-23, symbol Diode:BAT54C
- removed H1, H2, H3, H4: Threaded_Standoff, asl_footprints:standoff_nut, symbol asl_symbols:Threaded_Standoff
- removed J1: USB_C_Receptacle_USB2.0, asl_footprints:USB_C_Receptacle_GCT_USB4085, symbol asl_symbols:USB_C_Receptacle_USB2.0
- removed Q3: FDN340P, Package_TO_SOT_SMD:SOT-23, symbol asl_symbols:FDN340P
- removed R16: 330KΩ, Resistor_SMD:R_0805_2012Metric, symbol Device:R_Small_US
- removed S12: B3FS-1010P, asl_footprints:6mm_tactile_smd, symbol asl_symbols:B3FS-1010P
- removed U1: ATSAMD21G15A-A, Package_QFP:TQFP-48_7x7mm_P0.5mm, symbol MCU_Microchip_SAMD:ATSAMD21G15A-A
- removed U4: AP2112K-3.3, Package_TO_SOT_SMD:SOT-23-5, symbol asl_symbols:AP2112K-3.3
- removed U9: LTC4412xS6, Package_TO_SOT_SMD:TSOT-23-6, symbol Power_Management:LTC4412xS6
- removed Y1: Crystal, Crystal:Crystal_SMD_0603-2Pin_6.0x3.5mm, symbol Device:Crystal
- added D3: LED, LED_SMD:LED_0805_2012Metric, symbol Device:LED
- added L1: 10µH, Inductor_SMD:L_0805_2012Metric, symbol Device:L_Small
- added S12, S14, S15: Gateron Blue, Button_Switch_Keyboard:SW_Cherry_MX_1.00u_PCB, symbol imperializer-rescue:switch_momentary_2pin-asl_symbols-imperializer-rescue
- added U1: MAX1724, Package_TO_SOT_SMD:SOT-23-5, symbol asl_symbols_new:MAX1724
- added U10: ATSAMD21E15A-A, Package_QFP:TQFP-32_7x7mm_P0.8mm, symbol MCU_Microchip_SAMD:ATSAMD21E15A-A
- BT1: value Battery -> 2466
- J2: value SWD_connector -> SHF-105-01-L-D-SM
- R12: value 330KΩ -> 330Ω
- R14, R15: value 5.1KΩ -> 470Ω
- R18, R19, R20, R21: value 10KΩ -> 470Ω
- S1, S10, S11, S2, S3, S4, S5, S6, S7, S8, S9: value switch_momentary_2pin -> Gateron Blue
- U2, U3: value LTC-4727 -> LTC-4727JS
- U6, U7: value LTC-4727 -> LTC-4727JR
Connections:
- net BTN: now also U10.3 (PA02)
- net GND: now also BT1.2 (-), D1.3, D2.1 (K), D3.1 (K), S12.1, S12.2, U1.2 (GND), U10.10 (GND), U10.28 (GND); no longer R14.2, R15.2
- net IRQ: now also U10.7 (PA06)
- net KEYA: now also S14.1, S15.1
- net RST: now also U10.26 (~RESET)
- net SCL: now also U10.22 (PA23)
- net SDA: now also U10.21 (PA22)
- net SWCLK: now also U10.31 (PA30)
- net SWDIO: now also U10.32 (PA31)
- net VBATT: now also L1.1, U1.1 (BATT), U1.3 (SHDN); no longer C5.1, Q1.2 (S), R11.2
- net VIN: now also Q1.3 (D), U10.30 (VDDIN), U10.9 (VDDANA)
- net d: now also S14.2
- net e: now also S15.2
- net mode: now also U10.8 (PA07)
- net at R18.1: now also U10.17 (PA16)
- net at R19.1: now also U10.18 (PA17)
- net at R20.1: now also U10.19 (PA18)
- net at R21.1: now also U10.20 (PA19)
- net at C3.2: now also U10.29 (VDDCORE)
- net at R14.1: now also U10.15 (PA14)
- net at R15.1: now also U10.16 (PA15)
- net at D2.2 (A): now also R14.2
- new net: C5.1, Q1.2 (S), R11.2, U1.4 (OUT)
- new net: D3.2 (A), R15.2
- new net: L1.2, U1.5 (LX)
Other:
- moved on the sheet: BT1, C5, D1, D4, Q1, Q2, R11, R12, R13, R17, SW1
