File: pcb/unitron.kicad_pcb (KiCad board)
At the start: 2 copper layers, 80.3 x 155 mm, 79 parts, among them J1 Conn_01x10_Male, J2 Conn_01x10_Female, J3 Conn_01x10_Male, J4 Conn_01x10_Female, SW1 SPST, SW2 SW_SPST, SW3 RotaryEncoder_Switch, U1 LTC-4727JS, U2 LTC-4727JS, U3 AS1115-BSST, U4 QT_Py, U5 MCP73831, U6 LTC-4727JR, U7 LTC-4727JR, U8 AS1115-BSST

Commit message: pcb v1.14
Parts:
- removed the S1 at (135.3, 163.5)
- added D9: LED, LED_SMD:LED_0805_2012Metric, F.Cu at (137.0, 105.3)
- added G***: LOGO, LOGO, B.Cu at (80.8, 95.4)
- added LS1: Speaker, Buzzer_Beeper:Buzzer_12x9.5RM7.6, F.Cu at (71.0, 70.0)
- added R16: 10KΩ, Resistor_SMD:R_0805_2012Metric, B.Cu at (137.0, 68.0)
- added S5: Gateron Blue, Button_Switch_Keyboard:SW_Cherry_MX_1.00u_PCB, F.Cu at (135.3, 163.5)
- BT1: footprint Connector_PinHeader_2.54mm:PinHeader_1x02_P2.54mm_Vertical -> Connector_JST:JST_PH_S2B-PH-SM4-TB_1x02-1MP_P2.00mm_Horizontal
- moved kibuzzard-6260D7DE 27.0 mm to (85.0, 58.0)
- moved kibuzzard-6260D796 13.5 mm to (112.0, 58.0)
- moved kibuzzard-6260D976 13.5 mm to (98.5, 58.0)
- moved D8 4.30 mm to (140.5, 105.3)
- moved BT1 2.51 mm to (134.8, 69.2)
- moved SW1 2.00 mm to (138.7, 111.5), turned to 180 degrees
- moved D7 1.00 mm to (133.6, 67.2)
- renumbered R16 to R17, R17 to R18, R18 to R19, R19 to R20, R20 to R21, R21 to R22, R22 to R23, R23 to R24, S2 to S1, S3 to S2, S4 to S3, S5 to S4
Connections:
- BT1 pad 1: Net-(BT1-Pad1) -> /VBATT
- D7 pad 2: /VBATT -> Net-(D7-Pad2)
- SW1 pad 1: Net-(BT1-Pad1) -> Net-(D7-Pad2)
- SW2 pad 1: /mode -> Net-(SW2-Pad1)
- U4 pad 7: /BTN -> Net-(SW2-Pad1)
- U4 pad 8: /mode -> Net-(LS1-Pad2)
Routing:
- net /BTN: track 96.6 -> 0.00 mm
- net Net-(J2-Pad5): track 46.7 -> 130.5 mm, vias 0 -> 1
- net /mode: track 49.8 -> 0.00 mm
- net Net-(D7-Pad2): track 0.00 -> 49.3 mm
- net Net-(BT1-Pad1): track 46.2 -> 0.00 mm
- net Net-(D9-Pad2): track 0.00 -> 45.6 mm, vias 0 -> 1
- net Net-(LS1-Pad2): track 0.00 -> 35.2 mm, vias 0 -> 1
- net Net-(SW2-Pad1): track 0.00 -> 32.0 mm
- net /KEYA: track 161.1 -> 172.5 mm
- net Net-(D8-Pad2): track 35.2 -> 39.6 mm
- net /VBATT: track 57.7 -> 60.9 mm
- net Net-(D8-Pad1): track 39.9 -> 41.6 mm
- net /KEYB: track 197.6 -> 198.3 mm
- net GND: vias 3 -> 5
Other:
- outline, holes or cut-outs redrawn
- board text added: "Unitron v1.14"
- board text added: "v1.14"
- board text removed: "Unitron v1.13"
- board text removed: "v1.13"

Commit message: clean up directory for sharing
Parts:
- J1, J3: value Conn_01x10_Male -> TSM-116-01-T-SV
- S1, S10, S11, S12, S13, S14, S2, S3, S4, S5, S6, S7, S8, S9: value Gateron Blue -> Gateron green; footprint Button_Switch_Keyboard:SW_Cherry_MX_1.00u_PCB -> asl_footprints:SW_Cherry_MX_1.00u_PCB
- SW2: value SW_SPST -> M2012EA2W13
- SW3: value RotaryEncoder_Switch -> M2012EA2W13
- U4: value QT_Py -> 4900
- moved LS1 41.5 mm to (83.9, 109.4), turned to 180 degrees
- moved C3 39.8 mm to (135.4, 110.2)
- moved D7 39.8 mm to (139.0, 106.6)
- moved G*** 39.8 mm to (86.2, 134.8)
- moved H1 39.8 mm to (78.0, 119.4)
- moved H4 39.8 mm to (141.0, 119.4)
- moved R12 39.8 mm to (123.4, 107.4)
- moved R13 39.8 mm to (126.4, 105.4)
- moved R14 39.8 mm to (122.4, 111.4)
- moved R17 39.8 mm to (145.4, 107.4)
- moved R18 39.8 mm to (125.6, 110.4)
- moved R21 39.8 mm to (135.4, 106.4)
- moved S4 39.8 mm to (140.7, 183.9)
- moved S7 39.8 mm to (83.6, 183.9)
- moved S8 39.8 mm to (102.6, 183.9)
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- renumbered BT1 to BT2
Connections:
- LS1 pad 1: GND -> Net-(LS1-Pad1)
- LS1 pad 2: Net-(LS1-Pad2) -> GND
- U4 pad 8: Net-(LS1-Pad2) -> Net-(LS1-Pad1)
Routing:
- net Net-(LS1-Pad1): track 0.00 -> 35.2 mm, vias 0 -> 1
- net Net-(LS1-Pad2): track 35.2 -> 0.00 mm, vias 1 -> 0
Other:
- outline, holes or cut-outs redrawn
- board text added: "Lustig Labworks May 2022"
- board text removed: "Lustig Labworks April 2022"
