File: pcb/unitron.kicad_sch (KiCad schematic)
At the start: 71 parts, among them J1 Conn_01x10_Male, J2 Conn_01x10_Female, J3 Conn_01x10_Male, J4 Conn_01x10_Female, SW1 SPST, SW2 SW_SPST, SW3 RotaryEncoder_Switch, U1 LTC-4727JS, U2 LTC-4727JS, U3 AS1115-BSST, U4 QT_Py, U5 MCP73831, U6 LTC-4727JR, U7 LTC-4727JR, U8 AS1115-BSST

Commit message: pcb v1.14
Parts:
- removed S1: Gateron Blue, Button_Switch_Keyboard:SW_Cherry_MX_1.00u_PCB, symbol imperializer-rescue:switch_momentary_2pin-asl_symbols-imperializer-rescue
- added D9: LED, LED_SMD:LED_0805_2012Metric, symbol Device:LED
- added LS1: (no value), symbol Device:Speaker
- added R16: 10KΩ, Resistor_SMD:R_0805_2012Metric, symbol Device:R_Small_US
- added S5: Gateron Blue, Button_Switch_Keyboard:SW_Cherry_MX_1.00u_PCB, symbol imperializer-rescue:switch_momentary_2pin-asl_symbols-imperializer-rescue
- BT1: footprint Connector_PinHeader_2.54mm:PinHeader_1x02_P2.54mm_Vertical -> Connector_JST:JST_PH_S2B-PH-SM4-TB_1x02-1MP_P2.00mm_Horizontal
- renumbered R16 to R17, R17 to R18, R18 to R19, R19 to R20, R20 to R21, R21 to R22, R22 to R23, R23 to R24, S2 to S1, S3 to S2, S4 to S3, S5 to S4
Connections:
- net GND: now also D9.1 (K), LS1.1
- net IRQ_mcu: now also R14.2, U4.2 (A1)
- net KEYA: now also S5.1
- net VBATT: now also BT1.1 (+); no longer D7.2 (A)
- net at J2.5 (Pin_5), S11.2: now also S5.2
- net at SW1.1 (A): now also D7.2 (A); no longer BT1.1 (+)
- net at D7.1 (K), R13.1, R17.1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: now also R16.1
- net BTN: no longer names the net of U4.7 (TX)
- net BTN: now also SW2.1 (A)
- net mode: no longer names the net of U4.8 (RX)
- net mode: now also LS1.2; no longer SW2.1 (A)
- new net: D9.2 (A), R16.2
Other:
- moved on the sheet: C3, D8, R17, R21, SW2, U5

Commit message: clean up directory for sharing
Parts:
- J1, J3: value Conn_01x10_Male -> TSM-108-01-T-SV
- J2, J4: value Conn_01x10_Female -> SSW-108-01-T-S
- LS1: value (none) -> PK-11N40PQ; footprint (none) -> Buzzer_Beeper:Buzzer_12x9.5RM7.6
- S1, S10, S11, S12, S13, S14, S2, S3, S4, S5, S6, S7, S8, S9: value Gateron Blue -> Gateron green; footprint Button_Switch_Keyboard:SW_Cherry_MX_1.00u_PCB -> asl_footprints:SW_Cherry_MX_1.00u_PCB
- SW1: value SPST -> B12AP
- SW2: value SW_SPST -> M2012EA2W13
- SW3: value RotaryEncoder_Switch -> PEC11R-4215F-S0024
- U4: value QT_Py -> 4900
- renumbered BT1 to BT2
Connections:
- net GND: now also LS1.2; no longer LS1.1
- net at U4.8 (RX): now also LS1.1; no longer LS1.2
Other:
- moved on the sheet: LS1
